File: Hardware/Long/Qwiic_Shield_for_Teensy_Long.brd (EAGLE design)
At the start: 17.8 x 61 mm, 37 parts, among them J1 QWIIC_RA, J2 QWIIC_RA, J4 QWIIC_Vertical, J5 ALT PWR

Commit message: Long version routed
Parts:
- removed U$11: (no value), output:QWIIC0
- added J3: QWIIC_Vertical, SparkFun-Connectors:JST04_1MM_VERT
- added LOGO5: QWIIC_LOGO_5MM, SparkFun-Aesthetics:QWIIC_5MM
- LOGO2: value SFE_LOGO_FLAME.1_INCH -> SFE_LOGO_NAME_FLAME.1_INCH; device SparkFun-Aesthetics:SFE_LOGO_FLAME_.1 -> SparkFun-Aesthetics:SFE_LOGO_NAME_FLAME_.1
- U$9: device output:QWIIC0 -> output:#GND#0
- moved LOGO3 34.3 mm to (8.89, 58.4)
- moved U$9 32.1 mm to (13.9, 1.27), flipped to the bottom
- moved R4 9.90 mm to (4.09, 56.5)
- moved U$4 6.74 mm to (3.99, 9.53)
- moved D1_BP 6.63 mm to (3.99, 8.89), turned to 0 degrees
- moved LOGO2 5.92 mm to (8.89, 32.6)
- moved I2C 5.82 mm to (4.78, 54.8), turned to 90 degrees
- moved U$2 5.20 mm to (8.89, 33.6)
- moved U$13 4.83 mm to (8.89, 30.7)
- moved LOGO4 4.80 mm to (8.89, 28.8)
- moved U$1 4.25 mm to (4.72, 55.9), turned to 90 degrees
- moved LOGO1 4.09 mm to (8.89, 35.5)
- moved U$8 3.58 mm to (8.89, 26.9)
- moved R3 3.09 mm to (4.11, 52.8), turned to 270 degrees
- moved U$12 2.31 mm to (8.89, 29.6)
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Connections:
- net 3.3V: now also J3.2
- net GND: now also J3.1
- net SCL: now also J3.4
- net SDA: now also J3.3
Routing:
- net SCL: track 0.00 -> 70.0 mm, vias 0 -> 1
- net 3.3V: track 0.00 -> 68.4 mm, vias 0 -> 3
- net SDA: track 0.00 -> 66.5 mm, vias 0 -> 2
- net N$3: track 0.00 -> 5.13 mm
- net N$4: track 0.00 -> 4.62 mm
- net N$1: track 0.00 -> 3.37 mm, vias 0 -> 1
- net N$5: track 0.00 -> 3.28 mm
- net N$2: track 0.00 -> 3.23 mm, vias 0 -> 1
