File: Hardware/Extended/Qwiic_Shield_for_Teensy_Extended.brd (EAGLE design)
At the start: 17.8 x 61 mm, 38 parts, among them J1 QWIIC_RA, J2 QWIIC_RA, J3 QWIIC_Vertical, J4 QWIIC_Vertical, J5 ALT PWR

Commit message: Moving to "extended" product name
-Eagle file name change (and sub-folder)
-added silk to extended version
Parts:
- added U$11, U$16: (no value), output:EXTENDED0
Changed lines of the file:
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@@
 <drawing>
 <settings>
-<setting alwaysvectorfont="yes"/>
+<setting alwaysvectorfont="no"/>
 <setting verticaltext="up"/>
 </settings>
@@
 <element name="LOGO5" library="SparkFun-Aesthetics" package="QWIIC_5MM" value="QWIIC_LOGO_5MM" x="8.89" y="31.623" smashed="yes" rot="MR0"/>
 <element name="U$9" library="output" package="#GND#0" value="" x="13.9192" y="1.27" smashed="yes" rot="MR0"/>
+<element name="U$11" library="output" package="EXTENDED0" value="" x="8.89" y="25.2476" smashed="yes"/>
+<element name="U$16" library="output" package="EXTENDED0" value="" x="8.89" y="27.94" smashed="yes" rot="MR0"/>
 </elements>
 <signals>

Commit message: Library updates, name prefix fix, measures update
Parts:
- removed U$14: TEENSY-LONGNO_SILK, teensy_boards:TEENSY-LONG_NO_SILK
- added J6: ALT PWR, SparkFun-Connectors:1X02_NO_SILK
- J1: value QWIIC_RA -> TEENSY_EXTENDED; device SparkFun-Connectors:JST04_1MM_RA -> teensy_boards:TEENSY_EXTENDED_NO_SILK
- J3: value QWIIC_Vertical -> QWIIC_RA; device SparkFun-Connectors:JST04_1MM_VERT -> SparkFun-Connectors:JST04_1MM_RA
- J5: value ALT PWR -> QWIIC_Vertical; device SparkFun-Connectors:1X02_NO_SILK -> SparkFun-Connectors:JST04_1MM_VERT
- moved J2 50.8 mm to (8.89, 5.08), turned to 0 degrees
- moved J5 44.5 mm to (8.89, 53.3)
- moved J3 36.8 mm to (8.89, 55.9), turned to 180 degrees
- moved J4 34.3 mm to (8.89, 19.1), turned to 0 degrees
- moved J1 12.7 mm to (8.89, 17.8)
Connections:
- net 3.3V: now also J5.2; no longer J1.2
- net 3.3V_1: now also J1.3.3V@1; no longer U$14.3.3V@1
- net 3.3V_2: now also J1.3.3V@2; no longer U$14.3.3V@2
- net 5V: now also J1.5V; no longer U$14.5V
- net D+: now also J1.D+; no longer U$14.D+
- net D-: now also J1.D-; no longer U$14.D-
- net GND: now also J1.AGND, J1.GND, J1.GND1, J1.GND2, J1.GND3, J1.GND4, J6.1; no longer J1.1, U$14.AGND, U$14.GND, U$14.GND1, U$14.GND2, U$14.GND3, U$14.GND4
- net N$3: now also J1.3V; no longer U$14.3V
- net N$4: now also J6.2; no longer J5.2
- net N$5: now also J1.PROG; no longer U$14.PROG
- net SCL: now also J1.19, J5.4; no longer J1.4, U$14.19
- net SDA: now also J1.18, J5.3; no longer J1.3, U$14.18
- net VBAT: now also J1.VBAT; no longer U$14.VBAT
- net VIN: now also J1.VIN; no longer U$14.VIN
Changed lines of the file:
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@@
 <layer number="45" name="Holes" color="7" fill="1" visible="yes" active="yes"/>
 <layer number="46" name="Milling" color="3" fill="1" visible="no" active="yes"/>
-<layer number="47" name="Measures" color="7" fill="1" visible="no" active="yes"/>
+<layer number="47" name="Measures" color="7" fill="1" visible="yes" active="yes"/>
 <layer number="48" name="Document" color="7" fill="1" visible="no" active="yes"/>
 <layer number="49" name="Reference" color="7" fill="1" visible="yes" active="yes"/>
@@
 <dimension x1="9.271" y1="8.9408" x2="9.271" y2="0" x3="-2.54" y3="4.4704" textsize="1.27" layer="47" unit="inch" visible="yes"/>
 <dimension x1="9.271" y1="13.1064" x2="9.271" y2="0" x3="-7.747" y3="6.5532" textsize="1.27" layer="47" unit="inch" visible="yes"/>
+<dimension x1="8.89" y1="58.42" x2="0" y2="58.42" x3="4.445" y3="63.5" textsize="1.778" layer="47" unit="inch" visible="yes"/>
+<dimension x1="8.89" y1="41.91" x2="8.89" y2="0" x3="33.02" y3="20.955" textsize="1.778" layer="47" unit="inch" visible="yes"/>
+<dimension x1="8.9662" y1="21.5392" x2="8.89" y2="0" x3="24.1724" y3="10.71566875" textsize="1.778" layer="47" unit="inch" visible="yes"/>
 </plain>
 <attributes>
@@
 <attribute name="REV" value="" x="-12.7" y="-12.7" size="1.778" layer="27" display="off"/>
 </element>
-<element name="J1" library="SparkFun-Connectors" package="JST04_1MM_RA" value="QWIIC_RA" x="8.89" y="5.08" smashed="yes">
+<element name="J2" library="SparkFun-Connectors" package="JST04_1MM_RA" value="QWIIC_RA" x="8.89" y="5.08" smashed="yes">
 <attribute name="NAME" x="7.493" y="2.921" size="0.6096" layer="25" font="vector" ratio="20"/>
 <attribute name="PROD_ID" value="CONN-13694" x="8.89" y="5.08" size="1.778" layer="27" display="off"/>
 <attribute name="VALUE" x="7.239" y="1.778" size="0.6096" layer="27" font="vector" ratio="20"/>
 </element>
-<element name="J2" library="SparkFun-Connectors" package="JST04_1MM_RA" value="QWIIC_RA" x="8.89" y="55.88" smashed="yes" rot="R180">
+<element name="J3" library="SparkFun-Connectors" package="JST04_1MM_RA" value="QWIIC_RA" x="8.89" y="55.88" smashed="yes" rot="R180">
 <attribute name="NAME" x="10.287" y="58.039" size="0.6096" layer="25" font="vector" ratio="20" rot="R180"/>
 <attribute name="PROD_ID" value="CONN-13694" x="8.89" y="55.88" size="1.778" layer="27" rot="R180" display="off"/>
 <attribute name="VALUE" x="10.541" y="59.182" size="0.6096" layer="27" font="vector" ratio="20" rot="R180"/>
 </element>
-<element name="J4" library="SparkFun-Connectors" package="JST04_1MM_VERT" value="QWIIC_Vertical" x="8.89" y="53.34" smashed="yes" rot="R180">
+<element name="J5" library="SparkFun-Connectors" package="JST04_1MM_VERT" value="QWIIC_Vertical" x="8.89" y="53.34" smashed="yes" rot="R180">
 <attribute name="NAME" x="8.874" y="48.77366875" size="0.6096" layer="25" rot="R180"/>
 <attribute name="PROD_ID" value="CONN-14483" x="8.89" y="53.34" size="1.778" layer="27" rot="R180" display="off"/>
@@
 <element name="U$18" library="output" package="#SDA#0" value="" x="1.778" y="21.59" smashed="yes" rot="MR0"/>
 <element name="U$19" library="output" package="#SCL#0" value="" x="1.7526" y="19.0754" smashed="yes" rot="MR0"/>
-<element name="J5" library="SparkFun-Connectors" package="1X02_NO_SILK" value="ALT PWR" x="8.89" y="8.89" smashed="yes" rot="R180">
+<element name="J6" library="SparkFun-Connectors" package="1X02_NO_SILK" value="ALT PWR" x="8.89" y="8.89" smashed="yes" rot="R180">
 <attribute name="NAME" x="10.16" y="7.493" size="0.6096" layer="25" font="vector" ratio="20" rot="R180"/>
 <attribute name="VALUE" x="10.16" y="10.922" size="0.6096" layer="27" font="vector" ratio="20" rot="R180"/>
@@
 <element name="U$2" library="output" package="TEENSY0" value="" x="8.89" y="33.6042" smashed="yes" rot="MR0"/>
 <element name="U$12" library="output" package="SHIELD0" value="" x="8.89" y="29.6418" smashed="yes" rot="MR0"/>
-<element name="U$14" library="teensy_boards" package="TEENSY-LONG_NO_SILK" value="TEENSY-LONGNO_SILK" x="8.89" y="17.78" smashed="yes">
+<element name="J1" library="teensy_boards" package="TEENSY_EXTENDED_NO_SILK" value="TEENSY_EXTENDED" x="8.89" y="17.78" smashed="yes">
 <attribute name="NAME" x="8.89" y="35.814" size="0.6096" layer="25" font="vector" ratio="20" align="bottom-center"/>
 <attribute name="VALUE" x="8.89" y="-1.524" size="0.6096" layer="27" font="vector" ratio="20" align="top-center"/>
 </element>
-<element name="J3" library="SparkFun-Connectors" package="JST04_1MM_VERT" value="QWIIC_Vertical" x="8.89" y="19.05" smashed="yes">
+<element name="J4" library="SparkFun-Connectors" package="JST04_1MM_VERT" value="QWIIC_Vertical" x="8.89" y="19.05" smashed="yes">
 <attribute name="NAME" x="8.906" y="23.61633125" size="0.6096" layer="25"/>
 <attribute name="PROD_ID" value="CONN-14483" x="8.89" y="19.05" size="1.778" layer="27" display="off"/>
@@
 <signals>
 <signal name="GND">
-<contactref element="J4" pad="1"/>
+<contactref element="J5" pad="1"/>
+<contactref element="J3" pad="1"/>
 <contactref element="J2" pad="1"/>
-<contactref element="J1" pad="1"/>
 <polygon width="0.2032" layer="1" isolate="0.2032">
 <vertex x="0" y="0"/>
@@
 <vertex x="17.78" y="60.96"/>
 </polygon>
-<contactref element="J5" pad="1"/>
+<contactref element="J6" pad="1"/>
 <contactref element="S1" pad="3"/>
-<contactref element="U$14" pad="GND4"/>
-<contactref element="U$14" pad="GND2"/>
-<contactref element="U$14" pad="GND3"/>
-<contactref element="U$14" pad="GND1"/>
-<contactref element="U$14" pad="GND"/>
-<contactref element="U$14" pad="AGND"/>
-<contactref element="J3" pad="1"/>
+<contactref element="J1" pad="GND4"/>
+<contactref element="J1" pad="GND2"/>
+<contactref element="J1" pad="GND3"/>
+<contactref element="J1" pad="GND1"/>
+<contactref element="J1" pad="GND"/>
+<contactref element="J1" pad="AGND"/>
+<contactref element="J4" pad="1"/>
 <via x="7.366" y="6.477" extent="1-16" drill="0.381"/>
 <via x="7.4168" y="18.2118" extent="1-16" drill="0.381"/>
@@
 </signal>
 <signal name="3.3V">
-<contactref element="J1" pad="2"/>
 <contactref element="J2" pad="2"/>
-<contactref element="J4" pad="2"/>
+<contactref element="J3" pad="2"/>
+<contactref element="J5" pad="2"/>
 <contactref element="I2C" pad="2"/>
 <contactref element="3V3_ISO" pad="1"/>
 <contactref element="D1_BP" pad="2"/>
 <contactref element="D1" pad="C"/>
-<contactref element="J3" pad="2"/>
+<contactref element="J4" pad="2"/>
 <wire x1="9.39" y1="55.88" x2="9.39" y2="54.3306" width="0.508" layer="1"/>
 <wire x1="9.39" y1="54.3306" x2="9.39" y2="52.587" width="0.508" layer="1"/>
@@
 </signal>
 <signal name="SDA">
-<contactref element="J1" pad="3"/>
 <contactref element="J2" pad="3"/>
+<contactref element="J3" pad="3"/>
+<contactref element="J5" pad="3"/>
+<contactref element="R4" pad="1"/>
+<contactref element="J1" pad="18"/>
 <contactref element="J4" pad="3"/>
-<contactref element="R4" pad="1"/>
-<contactref element="U$14" pad="18"/>
-<contactref element="J3" pad="3"/>
 <wire x1="8.39" y1="55.88" x2="8.39" y2="52.587" width="0.254" layer="1"/>
 <wire x1="8.39" y1="52.587" x2="8.368" y2="52.565" width="0.254" layer="1"/>
@@
 </signal>
 <signal name="SCL">
-<contactref element="J1" pad="4"/>
 <contactref element="J2" pad="4"/>
+<contactref element="J3" pad="4"/>
+<contactref element="J5" pad="4"/>
+<contactref element="R3" pad="1"/>
+<contactref element="J1" pad="19"/>
 <contactref element="J4" pad="4"/>
-<contactref element="R3" pad="1"/>
-<contactref element="U$14" pad="19"/>
-<contactref element="J3" pad="4"/>
 <wire x1="7.39" y1="55.88" x2="7.39" y2="53.6448" width="0.254" layer="1"/>
 <wire x1="7.39" y1="53.6448" x2="7.39" y2="52.587" width="0.254" layer="1"/>
@@
 </signal>
 <signal name="N$4">
-<contactref element="J5" pad="2"/>
+<contactref element="J6" pad="2"/>
 <contactref element="D1_BP" pad="1"/>
 <contactref element="D1" pad="A"/>
@@
 <signal name="N$5">
 <contactref element="S1" pad="1"/>
-<contactref element="U$14" pad="PROG"/>
+<contactref element="J1" pad="PROG"/>
 <wire x1="6.35" y1="46.99" x2="6.35" y2="44.069" width="0.254" layer="1"/>
 <wire x1="6.35" y1="44.069" x2="6.096" y2="43.815" width="0.254" layer="1"/>
 </signal>
 <signal name="VBAT">
-<contactref element="U$14" pad="VBAT"/>
+<contactref element="J1" pad="VBAT"/>
 </signal>
 <signal name="VIN">
-<contactref element="U$14" pad="VIN"/>
+<contactref element="J1" pad="VIN"/>
 </signal>
 <signal name="N$3">
 <contactref element="3V3_ISO" pad="2"/>
-<contactref element="U$14" pad="3V"/>
+<contactref element="J1" pad="3V"/>
 <wire x1="5.0038" y1="4.2545" x2="5.0038" y2="5.1562" width="0.508" layer="16"/>
 <wire x1="5.0038" y1="5.1562" x2="3.81" y2="6.35" width="0.508" layer="16"/>
@@
 </signal>
 <signal name="5V">
-<contactref element="U$14" pad="5V"/>
+<contactref element="J1" pad="5V"/>
 </signal>
 <signal name="D+">
-<contactref element="U$14" pad="D+"/>
+<contactref element="J1" pad="D+"/>
 </signal>
 <signal name="D-">
-<contactref element="U$14" pad="D-"/>
+<contactref element="J1" pad="D-"/>
 </signal>
 <signal name="3.3V_2">
-<contactref element="U$14" pad="3.3V@2"/>
+<contactref element="J1" pad="3.3V@2"/>
 </signal>
 <signal name="3.3V_1">
-<contactref element="U$14" pad="3.3V@1"/>
+<contactref element="J1" pad="3.3V@1"/>
 </signal>
 </signals>
